Commit message: Macro for robot's wheels

File: nemo/models/robot/model.xacro (robot description, xacro)
@@ -3,6 +3,8 @@
     <model name="robot"
         xmlns:xacro="http://ros.org/wiki/xacro">
+        <!-- Xacro properties -->
         <xacro:property name="base_width" value="2.0"/>
         <xacro:property name="base_height" value="0.8"/>
+        <xacro:property name="wheel_radius" value="0.3"/>
         <static>false</static>
         <!-- Differential Drive Plugin -->
@@ -13,5 +15,5 @@
             <!-- Kinematics -->
             <wheel_separation>${base_width}</wheel_separation>
-            <wheel_radius>0.3</wheel_radius>
+            <wheel_radius>${wheel_radius}</wheel_radius>
             <!-- Output -->
             <odom_publish_frequency>2</odom_publish_frequency>
@@ -20,4 +22,6 @@
             <child_frame_id>base_link</child_frame_id>
         </plugin>
+        <!--Joint state publisher plugin -->
+        <plugin name="ignition::gazebo::systems::JointStatePublisher" filename="libignition-gazebo-joint-state-publisher-system.so"/>
         <!-- IMU Plugin -->
         <plugin name="ignition::gazebo::systems::Imu" filename="libignition-gazebo-imu-system.so"/>
@@ -26,8 +30,4 @@
             <render_engine>ogre2</render_engine>
         </plugin>
-        <!-- Lidar -->
-        <frame name="lidar_frame" attached_to='base_link'>
-            <pose>${base_width/2} 0 0.5 0 0 0</pose>
-        </frame>
         <!-- Chassis -->
         <link name='base_link'>
@@ -78,8 +78,101 @@
                 </geometry>
             </collision>
-            <sensor name='gpu_lidar' type='gpu_lidar'>"
-                <pose relative_to='lidar_frame'>0 0 0 0 0 0</pose>
-                <topic>lidar</topic>
-                <update_rate>10</update_rate>
+        </link>
+        <!-- Footprint -->
+        <link name="base_footprint"/>
+        <joint name="base_joint" type="fixed">
+            <parent>base_link</parent>
+            <child>base_footprint</child>
+        </joint>
+        <!-- Front wheels -->
+        <xacro:macro name="wheel" params="prefix x_reflect y_reflect">
+            <link name="${prefix}_wheel">
+                <pose>0.5 ${y_reflect*1.1} -0.2 ${pi/2} 0 0</pose>
+                <inertial>
+                    <mass>2</mass>
+                    <inertia>
+                        <ixx>0.145833</ixx>
+                        <ixy>0</ixy>
+                        <ixz>0</ixz>
+                        <iyy>0.145833</iyy>
+                        <iyz>0</iyz>
+                        <izz>0.125</izz>
+                    </inertia>
+                </inertial>
+                <visual name="visual">
+                    <geometry>
+                        <cylinder>
+                            <radius>${wheel_radius}</radius>
+                            <length>0.1</length>
+                        </cylinder>
+                    </geometry>
+                    <material>
+                        <ambient>0.2 0.2 0.2 1</ambient>
+                        <diffuse>0.2 0.2 0.2 1</diffuse>
+                        <specular>0.2 0.2 0.2 1</specular>
+                    </material>
+                </visual>
+                <collision name='collision'>
+                    <geometry>
+                        <cylinder>
+                            <radius>${wheel_radius}</radius>
+                            <length>0.1</length>
+                        </cylinder>
+                    </geometry>
+                </collision>
+            </link>
+            <joint name='${prefix}_wheel_joint' type='revolute'>
+                <pose relative_to='${prefix}_wheel'/>
+                <parent>base_link</parent>
+                <child>${prefix}_wheel</child>
+                <axis>
+                    <xyz expressed_in='__model__'>0 1 0</xyz>
+                    <limit>
+                        <lower>-1.79769e+308</lower>
+                        <upper>1.79769e+308</upper>
+                    </limit>
+                </axis>
+            </joint>
+        </xacro:macro>
+        <xacro:wheel prefix="left" x_reflect="-1" y_reflect="1" />
+        <xacro:wheel prefix="right" x_reflect="-1" y_reflect="-1" />
+        <!-- Caster wheel -->
+        <link name="caster_wheel">
+            <pose>-0.8 0 -0.4 0 0 0</pose>
+            <visual name='visual'>
+                <geometry>
+                    <sphere>
+                        <radius>0.1</radius>
+                    </sphere>
+                </geometry>
+                <material>
+                    <ambient>0.2 0.2 0.2 1</ambient>
+                    <diffuse>0.2 0.2 0.2 1</diffuse>
+                    <specular>0.2 0.2 0.2 1</specular>
+                </material>
+            </visual>
+            <collision name='collision'>
+                <geometry>
+                    <sphere>
+                        <radius>0.1</radius>
+                    </sphere>
+                </geometry>
+            </collision>
+        </link>
+        <joint name="caster_wheel_joint" type="fixed">
+            <parent>base_link</parent>
+            <child>caster_wheel</child>
+            <axis>
+                <xyz>0.24 0 0</xyz>
+                <limit>
+                    <lower>-1.79769e+308</lower>
+                    <upper>1.79769e+308</upper>
+                </limit>
+            </axis>
+        </joint>
+        <!-- LiDAR -->
+        <link name="lidar_link">
+            <pose>${base_width/2} 0 0.5 0 0 0</pose>
+            <sensor name='gpu_lidar' type='gpu_lidar'>
                 <ray>
                     <scan>
@@ -104,137 +197,14 @@
                 </ray>
                 <always_on>1</always_on>
+                <update_rate>30</update_rate>
                 <visualize>true</visualize>
+                <topic>lidar</topic>
             </sensor>
         </link>
-        <!-- Footprint -->
-        <link name="base_footprint"/>
-        <joint name="base_joint" type="fixed">
-            <parent>base_link</parent>
-            <child>base_footprint</child>
-        </joint>
-        <!-- Left Wheel -->
-        <link name='left_wheel'>
-            <pose>0.5 1.1 -0.2 ${pi/2} 0 0</pose>
-            <inertial>
-                <mass>2</mass>
-                <inertia>
-                    <ixx>0.145833</ixx>
-                    <ixy>0</ixy>
-                    <ixz>0</ixz>
-                    <iyy>0.145833</iyy>
-                    <iyz>0</iyz>
-                    <izz>0.125</izz>
-                </inertia>
-            </inertial>
-            <visual name='visual'>
-                <geometry>
-                    <cylinder>
-                        <radius>0.3</radius>
-                        <length>0.1</length>
-                    </cylinder>
-                </geometry>
-                <material>
-                    <ambient>0.2 0.2 0.2 1</ambient>
-                    <diffuse>0.2 0.2 0.2 1</diffuse>
-                    <specular>0.2 0.2 0.2 1</specular>
-                </material>
-            </visual>
-            <collision name='collision'>
-                <geometry>
-                    <cylinder>
-                        <radius>0.3</radius>
-                        <length>0.1</length>
-                    </cylinder>
-                </geometry>
-            </collision>
-        </link>
-        <joint name='left_wheel_joint' type='revolute'>
-            <pose relative_to='left_wheel'/>
-            <parent>base_link</parent>
-            <child>left_wheel</child>
+        <joint name="lidar_joint" type="fixed">
+            <parent>base_link</parent>
+            <child>lidar_link</child>
             <axis>
-                <xyz expressed_in='__model__'>0 1 0</xyz>
-                <limit>
-                    <lower>-1.79769e+308</lower>
-                    <upper>1.79769e+308</upper>
-                </limit>
-            </axis>
-        </joint>
-        <!-- Right Wheel -->
-        <link name='right_wheel'>
-            <pose>0.5 -1.1 -0.2 ${pi/2} 0 0</pose>
-            <inertial>
-                <mass>2</mass>
-                <inertia>
-                    <ixx>0.145833</ixx>
-                    <ixy>0</ixy>
-                    <ixz>0</ixz>
-                    <iyy>0.145833</iyy>
-                    <iyz>0</iyz>
-                    <izz>0.125</izz>
-                </inertia>
-            </inertial>
-            <visual name='visual'>
-                <geometry>
-                    <cylinder>
-                        <radius>0.3</radius>
-                        <length>0.1</length>
-                    </cylinder>
-                </geometry>
-                <material>
-                    <ambient>0.2 0.2 0.2 1</ambient>
-                    <diffuse>0.2 0.2 0.2 1</diffuse>
-                    <specular>0.2 0.2 0.2 1</specular>
-                </material>
-            </visual>
-            <collision name='collision'>
-                <geometry>
-                    <cylinder>
-                        <radius>0.3</radius>
-                        <length>0.1</length>
-                    </cylinder>
-                </geometry>
-            </collision>
-        </link>
-        <joint name='right_wheel_joint' type='revolute'>
-            <pose relative_to='right_wheel'/>
-            <parent>base_link</parent>
-            <child>right_wheel</child>
-            <axis>
-                <xyz expressed_in='__model__'>0 1 0</xyz>
-                <limit>
-                    <lower>-1.79769e+308</lower>
-                    <upper>1.79769e+308</upper>
-                </limit>
-            </axis>
-        </joint>
-        <!-- Caster wheel -->
-        <link name="caster_wheel">
-            <pose>-0.8 0 -0.4 0 0 0</pose>
-            <visual name='visual'>
-                <geometry>
-                    <sphere>
-                        <radius>0.1</radius>
-                    </sphere>
-                </geometry>
-                <material>
-                    <ambient>0.2 0.2 0.2 1</ambient>
-                    <diffuse>0.2 0.2 0.2 1</diffuse>
-                    <specular>0.2 0.2 0.2 1</specular>
-                </material>
-            </visual>
-            <collision name='collision'>
-                <geometry>
-                    <sphere>
-                        <radius>0.1</radius>
-                    </sphere>
-                </geometry>
-            </collision>
-        </link>
-        <joint name="caster_wheel_joint" type="fixed">
-            <parent>base_link</parent>
-            <child>caster_wheel</child>
-            <axis>
-                <xyz>0.24 0 0</xyz>
+                <xyz>0 0.5 0</xyz>
                 <limit>
                     <lower>-1.79769e+308</lower>

Commit message: Using nav2_bringup for launch

File: nemo/models/robot/model.xacro (robot description, xacro)
@@ -140,4 +140,15 @@
         <link name="caster_wheel">
             <pose>-0.8 0 -0.4 0 0 0</pose>
+            <inertial>
+                <mass>2</mass>
+                <inertia>
+                    <ixx>0.145833</ixx>
+                    <ixy>0</ixy>
+                    <ixz>0</ixz>
+                    <iyy>0.145833</iyy>
+                    <iyz>0</iyz>
+                    <izz>0.125</izz>
+                </inertia>
+            </inertial>
             <visual name='visual'>
                 <geometry>
@@ -174,5 +185,5 @@
         <link name="lidar_link">
             <pose>${base_width/2} 0 0.5 0 0 0</pose>
-            <sensor name='gpu_lidar' type='gpu_lidar'>
+            <sensor name='scan' type='gpu_lidar'>
                 <ray>
                     <scan>
